File: PCB/buckConv.sch (KiCad schematic (older format))
At the start: 11 parts

Commit message: Schematic one step closer
Parts:
- C10, C11, C12, C13, C14, C9: renamed from C?; footprint (none) -> Capacitors_SMD:C_0805
- D5: renamed from D?; footprint (none) -> Diodes_SMD:D_SOD-323
- L1: renamed from L?; footprint (none) -> myStuff:cc_5022
- gave numbers to parts that had none: 3
Connections:
- wire segments 55 -> 36
Changed lines of the file:
@@
 EESchema Schematic File Version 2
+LIBS:veloGen-rescue
 LIBS:power
 LIBS:device
@@
 LIBS:contrib
 LIBS:valves
+LIBS:myStuff
 LIBS:veloGen-cache
 EELAYER 26 0
@@
 $EndDescr
 $Comp
-L C C?
+L C C10
 U 1 1 58D19908
 P 3450 3250
-F 0 "C?" H 3550 3150 50  0000 L CNN
+F 0 "C10" H 3550 3150 50  0000 L CNN
 F 1 "10u" H 3550 3050 50  0000 L CNN
-F 2 "" H 3488 3100 50  0001 C CNN
+F 2 "Capacitors_SMD:C_0805" H 3488 3100 50  0001 C CNN
 F 3 "" H 3450 3250 50  0001 C CNN
 	1    3450 3250
@@
 $EndComp
 $Comp
-L L L?
+L L L1
 U 1 1 58D1990A
 P 4950 2500
-F 0 "L?" V 5140 2500 50  0000 C CNN
+F 0 "L1" V 5140 2500 50  0000 C CNN
 F 1 "L" V 5049 2500 50  0000 C CNN
-F 2 "" H 4950 2500 50  0001 C CNN
+F 2 "myStuff:cc_5022" H 4950 2500 50  0001 C CNN
 F 3 "" H 4950 2500 50  0001 C CNN
 	1    4950 2500
@@
 $EndComp
 $Comp
-L D_Schottky D?
+L D_Schottky D6
 U 1 1 58D1990B
 P 4700 3200
-F 0 "D?" H 4900 3100 50  0000 L CNN
+F 0 "D6" H 4900 3100 50  0000 L CNN
 F 1 "STPS3L40UF" H 4350 3100 50  0000 L CNN
 F 2 "Diodes_SMD:D_SMB_Standard" H 4700 3200 50  0001 C CNN
@@
 $EndComp
 $Comp
-L C C?
+L C C14
 U 1 1 58D1990C
 P 5550 3250
-F 0 "C?" H 5600 3150 50  0000 L CNN
+F 0 "C14" H 5600 3150 50  0000 L CNN
 F 1 "10u" H 5600 3050 50  0000 L CNN
-F 2 "" H 5588 3100 50  0001 C CNN
+F 2 "Capacitors_SMD:C_0805" H 5588 3100 50  0001 C CNN
 F 3 "" H 5550 3250 50  0001 C CNN
 	1    5550 3250
@@
 $EndComp
 $Comp
-L STL6N3LLH6 Q?
+L STL6N3LLH6 Q3
 U 1 1 58D19914
 P 4300 2600
-F 0 "Q?" V 4643 2600 50  0000 C CNN
+F 0 "Q3" V 4643 2600 50  0000 C CNN
 F 1 "STL6N3LLH6" V 4552 2600 50  0000 C CNN
 F 2 "myStuff:PowerFLAT_2x2" H 4550 2500 50  0001 L CIN
@@
 $EndComp
 $Comp
-L C C?
+L C C9
 U 1 1 58D19918
 P 2450 4450
-F 0 "C?" H 2400 4350 50  0000 R CNN
+F 0 "C9" H 2400 4350 50  0000 R CNN
 F 1 "470n" H 2400 4550 50  0000 R CNN
-F 2 "" H 2488 4300 50  0001 C CNN
+F 2 "Capacitors_SMD:C_0805" H 2488 4300 50  0001 C CNN
 F 3 "" H 2450 4450 50  0001 C CNN
 	1    2450 4450
@@
 $EndComp
 $Comp
-L GND #PWR?
+L GND #PWR022
 U 1 1 58D19919
 P 2600 4650
-F 0 "#PWR?" H 2600 4400 50  0001 C CNN
+F 0 "#PWR022" H 2600 4400 50  0001 C CNN
 F 1 "GND" H 2450 4600 50  0000 C CNN
 F 2 "" H 2600 4650 50  0001 C CNN
@@
 $EndComp
 $Comp
-L C C?
+L C C12
 U 1 1 58D1991A
 P 3800 4300
-F 0 "C?" H 3685 4254 50  0000 R CNN
+F 0 "C12" H 3685 4254 50  0000 R CNN
 F 1 "470n" H 3650 4350 50  0000 R CNN
-F 2 "" H 3838 4150 50  0001 C CNN
+F 2 "Capacitors_SMD:C_0805" H 3838 4150 50  0001 C CNN
 F 3 "" H 3800 4300 50  0001 C CNN
 	1    3800 4300
@@
 $EndComp
 $Comp
-L D_Schottky D?
+L D_Schottky D5
 U 1 1 58D1991B
 P 3150 4050
-F 0 "D?" H 3250 3950 50  0000 L CNN
+F 0 "D5" H 3250 3950 50  0000 L CNN
 F 1 "B5819WS" V 3195 4129 50  0001 L CNN
-F 2 "" H 3150 4050 50  0001 C CNN
+F 2 "Diodes_SMD:D_SOD-323" H 3150 4050 50  0001 C CNN
 F 3 "" H 3150 4050 50  0001 C CNN
 	1    3150 4050
@@
 $EndComp
 $Comp
-L LTC4440 U?
+L LTC4440 U5
 U 1 1 58D1991C
 P 2950 4550
-F 0 "U?" H 3050 4500 60  0000 C CNN
+F 0 "U5" H 3050 4500 60  0000 C CNN
 F 1 "LTC4440-5" H 3150 4400 60  0000 C CNN
 F 2 "TO_SOT_Packages_SMD:SOT-23-6_Handsoldering" H 3750 4350 60  0001 C CNN
@@
 $EndComp
 Wire Wire Line
-	1600 3550 3450 3550
-Wire Wire Line
-	3450 3550 3800 3550
-Wire Wire Line
-	3800 3550 4700 3550
-Wire Wire Line
-	4700 3550 5250 3550
-Wire Wire Line
-	5250 3550 5550 3550
-Wire Wire Line
-	5550 3550 8200 3550
+	1600 3550 8200 3550
 Wire Wire Line
 	3450 2500 3450 3100
@@
 Connection ~ 3450 2500
 Wire Wire Line
-	4500 2500 4550 2500
-Wire Wire Line
-	4550 2500 4700 2500
-Wire Wire Line
-	4700 2500 4800 2500
+	4500 2500 4800 2500
 Wire Wire Line
 	4700 3550 4700 3350
 Connection ~ 3450 3550
 Wire Wire Line
-	1600 2500 3450 2500
-Wire Wire Line
-	3450 2500 3800 2500
-Wire Wire Line
-	3800 2500 4100 2500
+	1600 2500 4100 2500
 Wire Wire Line
 	4700 2500 4700 3050
 Connection ~ 4700 2500
 Wire Wire Line
-	5550 3100 5550 2500
-Wire Wire Line
-	5100 2500 5250 2500
-Wire Wire Line
-	5250 2500 5550 2500
-Wire Wire Line
-	5550 2500 5800 2500
-Wire Wire Line
-	5800 2500 8050 2500
-Wire Wire Line
-	8050 2500 8200 2500
+	5550 2500 5550 3100
+Wire Wire Line
+	5100 2500 8200 2500
 Wire Wire Line
 	5550 3550 5550 3400
@@
 Connection ~ 5550 2500
 Wire Wire Line
-	2450 4300 2600 4300
-Wire Wire Line
-	2600 4300 2750 4300
-Wire Wire Line
-	2600 4400 2600 4600
-Wire Wire Line
-	2600 4600 2600 4650
+	2450 4300 2750 4300
+Wire Wire Line
+	2600 4400 2600 4650
 Wire Wire Line
 	2600 4400 2750 4400
@@
 	3000 4050 2600 4050
 Wire Wire Line
-	2600 3850 2600 4050
-Wire Wire Line
-	2600 4050 2600 4300
+	2600 3850 2600 4300
 Connection ~ 2600 4300
 Wire Wire Line
@@
 	3600 4050 3600 4300
 Wire Wire Line
-	3550 4300 3600 4300
-Wire Wire Line
-	3600 4300 3650 4300
+	3550 4300 3650 4300
 Connection ~ 3600 4300
 Wire Wire Line
-	3550 4500 4000 4500
-Wire Wire Line
-	4000 4500 4350 4500
+	3550 4500 4350 4500
 Wire Wire Line
 	3550 4400 4300 4400
@@
 	1600 4950 2750 4950
 $Comp
-L GND #PWR?
+L GND #PWR023
 U 1 1 58D19CF5
 P 4000 3650
-F 0 "#PWR?" H 4000 3400 50  0001 C CNN
+F 0 "#PWR023" H 4000 3400 50  0001 C CNN
 F 1 "GND" H 3850 3550 50  0000 C CNN
 F 2 "" H 4000 3650 50  0001 C CNN
@@
 Connection ~ 5800 2500
 $Comp
-L PWR_FLAG #FLG?
-U 1 1 58D1D6FC
-P 8050 2450
-F 0 "#FLG?" H 8050 2525 50  0001 C CNN
-F 1 "PWR_FLAG" H 8050 2624 50  0000 C CNN
-F 2 "" H 8050 2450 50  0000 C CNN
-F 3 "" H 8050 2450 50  0000 C CNN
-	1    8050 2450
-	1    0    0    -1
-$EndComp
-Wire Wire Line
-	8050 2450 8050 2500
-Connection ~ 8050 2500
-$Comp
-L C C?
+L C C13
 U 1 1 58D2C0CB
 P 5250 3250
-F 0 "C?" H 5200 3350 50  0000 R CNN
+F 0 "C13" H 5200 3350 50  0000 R CNN
 F 1 "470n" H 5200 3450 50  0000 R CNN
-F 2 "" H 5288 3100 50  0001 C CNN
+F 2 "Capacitors_SMD:C_0805" H 5288 3100 50  0001 C CNN
 F 3 "" H 5250 3250 50  0001 C CNN
 	1    5250 3250
@@
 Connection ~ 5250 2500
 $Comp
-L C C?
+L C C11
 U 1 1 58D2C50B
 P 3800 3250
-F 0 "C?" H 3750 3350 50  0000 R CNN
+F 0 "C11" H 3750 3350 50  0000 R CNN
 F 1 "470n" H 3750 3450 50  0000 R CNN
-F 2 "" H 3838 3100 50  0001 C CNN
+F 2 "Capacitors_SMD:C_0805" H 3838 3100 50  0001 C CNN
 F 3 "" H 3800 3250 50  0001 C CNN
 	1    3800 3250

Commit message: Layout ideas
Parts:
- added R14: 470, Resistors_SMD:R_0805, symbol R
- L1: value L -> 68u; footprint myStuff:cc_5022 -> myStuff:MSS1048
Connections:
- wire segments 36 -> 37
Changed lines of the file:
@@
 P 4950 2500
 F 0 "L1" V 5140 2500 50  0000 C CNN
-F 1 "L" V 5049 2500 50  0000 C CNN
-F 2 "myStuff:cc_5022" H 4950 2500 50  0001 C CNN
-F 3 "" H 4950 2500 50  0001 C CNN
+F 1 "68u" V 5049 2500 50  0000 C CNN
+F 2 "myStuff:MSS1048" H 4950 2500 50  0001 C CNN
+F 3 "http://www.coilcraft.com/pdfs/mss1048.pdf" H 4950 2500 50  0001 C CNN
 	1    4950 2500
 	0    -1   -1   0
@@
 $EndComp
 $Comp
-L GND #PWR022
+L GND #PWR20
 U 1 1 58D19919
 P 2600 4650
-F 0 "#PWR022" H 2600 4400 50  0001 C CNN
+F 0 "#PWR20" H 2600 4400 50  0001 C CNN
 F 1 "GND" H 2450 4600 50  0000 C CNN
 F 2 "" H 2600 4650 50  0001 C CNN
@@
 Wire Wire Line
 	3550 4400 4300 4400
-Wire Wire Line
-	4300 4400 4300 2800
 Connection ~ 4550 2500
 Wire Wire Line
@@
 	1600 4950 2750 4950
 $Comp
-L GND #PWR023
+L GND #PWR21
 U 1 1 58D19CF5
 P 4000 3650
-F 0 "#PWR023" H 4000 3400 50  0001 C CNN
+F 0 "#PWR21" H 4000 3400 50  0001 C CNN
 F 1 "GND" H 3850 3550 50  0000 C CNN
 F 2 "" H 4000 3650 50  0001 C CNN
@@
 	3800 3100 3800 2500
 Connection ~ 3800 2500
+$Comp
+L R R14
+U 1 1 58D4E6F9
+P 4300 3150
+F 0 "R14" H 4370 3196 50  0000 L CNN
+F 1 "470" H 4370 3105 50  0000 L CNN
+F 2 "Resistors_SMD:R_0805" V 4230 3150 50  0001 C CNN
+F 3 "" H 4300 3150 50  0001 C CNN
+	1    4300 3150
+	1    0    0    -1
+$EndComp
+Wire Wire Line
+	4300 3000 4300 2800
+Wire Wire Line
+	4300 4400 4300 3300
 $EndSCHEMATC

Commit message: Added SEPIC ltspice model
Parts:
- removed C12, C9: 470n, Capacitors_SMD:C_0805, symbol C
- removed D5: B5819WS, Diodes_SMD:D_SOD-323, symbol D_Schottky
- removed L1: 68u, myStuff:MSS1048, symbol L
- removed R14: 470, Resistors_SMD:R_0805, symbol R
- removed U5: LTC4440-5, TO_SOT_Packages_SMD:SOT-23-6_Handsoldering, symbol LTC4440
- added C15: 470n, Capacitors_SMD:C_0805, symbol C
- added R15: 10R, Resistors_SMD:R_0805_HandSoldering, symbol R
- added R16, R17: 0.11R, symbol R
- added T1: 10u 10u k=0.99, symbol Transformer_1P_1S
- added U5: MCP1630, Housings_SSOP:MSOP-8_3x3mm_Pitch0.65mm, symbol MCP1630
- C13: value 470n -> 1u; footprint Capacitors_SMD:C_0805 -> (none)
Connections:
- net labels added: +BATT
- wire segments 37 -> 31
Other:
- note added: "When buckPwm is high, Vext is forced low\nOn neg. edge: Vext high until cycle current limit kicks in\n ... or until buckPwm goes high again"
- moved on the sheet: C10, C11, D6

Commit message: Schematic work
Parts:
- added C?: ?, Capacitors_SMD:C_0805, symbol C
- added R? (x2): ?, Resistors_SMD:R_0805_HandSoldering, symbol R
Connections:
- net labels added: maxSwCurr
- wire segments 31 -> 46
Other:
- note added: "0.9 V max."
- note added: "EA. becomes\nvoltage follower"
- note added: "When buckPwm is high, Vext is forced low\nOn neg. edge: Vext goes high until cycle \ncurrent limit kicks in\n ... or until buckPwm goes high again"
- note added: "maxSwCurr defines the cycle by\ncycle current limit threshold\nNeeds to connect to a DAC (2.7V max.)"
- note removed: "When buckPwm is high, Vext is forced low\nOn neg. edge: Vext high until cycle current limit kicks in\n ... or until buckPwm goes high again"
- moved on the sheet: R16, R17
