File: PCB/sepicConv.sch (KiCad schematic (older format))
At the start: 19 parts, among them Q3 STL6N3LLH6, T1 MSD1260, U5 MCP1630

Commit message: built first prototype, some mods are needed
Parts:
- C3: value 47n -> 2u2
Changed lines of the file:
@@
-EESchema Schematic File Version 2
+EESchema Schematic File Version 3
 LIBS:veloGen-rescue
 LIBS:power
@@
 LIBS:contrib
 LIBS:valves
-LIBS:myStuff
 LIBS:veloGen-cache
 EELAYER 26 0
@@
 P 3100 2100
 F 0 "C3" H 2950 1900 50  0000 L CNN
-F 1 "47n" H 2950 1800 50  0000 L CNN
+F 1 "2u2" H 2950 1800 50  0000 L CNN
 F 2 "Capacitors_SMD:C_0805" H 3138 1950 50  0001 C CNN
 F 3 "" H 3100 2100 50  0001 C CNN
