File: PCB2/velogen2.kicad_pcb (KiCad board)
At the start: 2 copper layers, 35 x 70 mm, 34 parts, among them J1 DYN, J2 Conn_01x05_Male, J3 AUX0, J4 AUX1, J5 AUX2, J6 BAT, Q1 BSS123, Q2 DMP10H400SE, SW1 SW_SPST, U1 DCDC_mod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

Commit message: PCB: Moved R2
Parts:
- added D6: B5819WS, Diode_SMD:D_SOD-323, F.Cu at (162.9, 41.6)
- added D7: B5819WS, Diode_SMD:D_SOD-323, F.Cu at (167.2, 41.6)
- moved R5 5.43 mm to (179.1, 67.3)
- moved R2 3.70 mm to (167.6, 78.7)
- moved C2 1.27 mm to (167.0, 74.9)
Connections:
- U2 pad 17: (no net) -> Net-(U2-Pad17)
- U2 pad 18: (no net) -> Net-(U2-Pad18)
- U2 pad 19: (no net) -> Net-(U2-Pad19)
- U2 pad 20: (no net) -> Net-(U2-Pad20)
- U2 pad 21: (no net) -> Net-(U2-Pad21)
- U2 pad 22: (no net) -> Net-(U2-Pad22)
- U2 pad 28: (no net) -> Net-(U2-Pad28)
- U2 pad 30: (no net) -> Net-(U2-Pad30)
- U2 pad 31: (no net) -> Net-(U2-Pad31)
- U2 pad 32: (no net) -> Net-(U2-Pad32)
- U2 pad 4: (no net) -> Net-(U2-Pad4)
- U2 pad 5: (no net) -> Net-(U2-Pad5)
- U2 pad 6: (no net) -> Net-(U2-Pad6)
- U2 pad 7: (no net) -> Net-(U2-Pad7)

Commit message: clean up schematic symbols
  * re-associate standard symbols with the standard library (needs to be
    installed)
  * remove `myStuff` library. Symbols from there are now in rescue.lib
  * make the 3V3 enable switch a jumper poking out trough the case
Parts:
- SW1: footprint Connector_JST:JST_EH_B2B-EH-A_1x02_P2.50mm_Vertical -> Connector_PinHeader_2.54mm:PinHeader_1x02_P2.54mm_Horizontal
Connections:
- U2 pad 17: Net-(U2-Pad17) -> (no net)
- U2 pad 18: Net-(U2-Pad18) -> (no net)
- U2 pad 19: Net-(U2-Pad19) -> (no net)
- U2 pad 20: Net-(U2-Pad20) -> (no net)
- U2 pad 21: Net-(U2-Pad21) -> (no net)
- U2 pad 22: Net-(U2-Pad22) -> (no net)
- U2 pad 28: Net-(U2-Pad28) -> (no net)
- U2 pad 30: Net-(U2-Pad30) -> (no net)
- U2 pad 31: Net-(U2-Pad31) -> (no net)
- U2 pad 32: Net-(U2-Pad32) -> (no net)
- U2 pad 4: Net-(U2-Pad4) -> (no net)
- U2 pad 5: Net-(U2-Pad5) -> (no net)
- U2 pad 6: Net-(U2-Pad6) -> (no net)
- U2 pad 7: Net-(U2-Pad7) -> (no net)

Commit message: move all small components to top side
Parts:
- C1, C2, C4, D5, R1, R2, R4, R5, R7, U3: moved to F.Cu
- Q1: value BSS123 -> BSS138
- SW1: moved to B.Cu
- moved D7 50.8 mm to (182.2, 90.2)
- moved D6 49.9 mm to (182.2, 87.6), turned to 180 degrees
- moved SW1 46.7 mm to (190.5, 90.2), turned to 0 degrees
- moved C2 44.4 mm to (177.2, 118.1)
- moved C3 9.61 mm to (170.8, 62.2), turned to 180 degrees
- moved D5 7.10 mm to (167.6, 82.5), turned to 90 degrees
- moved R1 7.10 mm to (170.2, 82.5), turned to 90 degrees
- moved R3 5.71 mm to (164.5, 87.6), turned to 180 degrees
- moved R5 5.24 mm to (184.2, 68.6), turned to 270 degrees
- moved C4 4.62 mm to (165.7, 62.9), turned to 0 degrees
- moved R2 4.07 mm to (164.5, 81.3), turned to 180 degrees
- moved Q1 4.07 mm to (164.5, 84.5), turned to 180 degrees
- moved U3 4.02 mm to (176.5, 64.8)
- moved R6 3.86 mm to (178.4, 88.9)
- moved R4 3.70 mm to (170.8, 66.0), turned to 90 degrees
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
Commit message: sch: fix some component names
Parts:
- D1, D2, D3, D4: value SS32 -> SS310
- Q1: value BSS138 -> BSS123
- SW1: value SW_SPST -> JMP

Commit message: put propper package (SMA) for diodes
Parts:
- D1, D2, D3, D4: footprint Diode_SMD:D_SMC -> Diode_SMD:D_SMA
- moved SW1 23.6 mm to (167.0, 87.6), turned to 180 degrees
- moved U1 10.8 mm to (172.7, 79.4), turned to 180 degrees
- moved R3 5.43 mm to (169.5, 85.7), turned to 270 degrees
- moved D5 4.45 mm to (172.1, 82.5)
- moved C1 3.86 mm to (186.1, 85.1)
- moved D6 3.86 mm to (182.9, 83.8)
- moved D7 3.86 mm to (182.9, 86.4)
- moved R6 3.86 mm to (179.1, 85.1)
- moved D3 3.42 mm to (178.4, 79.4)
- moved D4 3.24 mm to (187.3, 79.4)
- moved Q1 1.91 mm to (166.4, 84.5)
- moved Q2 1.91 mm to (168.9, 76.2)
- moved R2 1.91 mm to (166.4, 81.3)
- moved D1 1.80 mm to (178.4, 74.3)
- moved D2 1.42 mm to (187.3, 74.3)
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Connections:
- SW1 pad 1: Net-(SW1-Pad1) -> GND
- SW1 pad 2: GND -> Net-(SW1-Pad2)
- U1 pad 4: Net-(SW1-Pad1) -> Net-(SW1-Pad2)

Commit message: did some routing of the power rails
  * kinda stuck on the 3V3, might need to re-consider placement
Parts:
- moved R5 35.5 mm to (169.5, 101.0), turned to 0 degrees
- moved J1 23.5 mm to (164.5, 66.0)
- moved J6 23.5 mm to (188.0, 66.0)
- moved C4 23.5 mm to (189.2, 62.9)
- moved Q1 22.7 mm to (188.6, 88.9)
- moved R2 22.7 mm to (188.6, 85.7)
- moved R3 22.5 mm to (191.8, 88.9), turned to 90 degrees
- moved R1 22.2 mm to (189.9, 73.0), turned to 180 degrees
- moved Q2 18.9 mm to (187.3, 80.6)
- moved D5 18.5 mm to (189.2, 75.6), turned to 180 degrees
- moved D2 18.4 mm to (168.9, 74.3), turned to 180 degrees
- moved D4 18.4 mm to (168.9, 79.4), turned to 180 degrees
- moved R4 14.1 mm to (184.8, 64.1), turned to 270 degrees
- moved U1 10.0 mm to (178.4, 87.6)
- moved R6 5.43 mm to (174.0, 83.2)
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Connections:
- J1 pad 1: Net-(D1-Pad2) -> Net-(D3-Pad2)
- J1 pad 2: Net-(D3-Pad2) -> Net-(D1-Pad2)
Routing:
- net +BATT: track 0.00 -> 34.3 mm, vias 0 -> 7
- net Net-(D3-Pad2): track 0.00 -> 33.2 mm, vias 0 -> 4
- net Net-(D5-Pad2): track 0.00 -> 21.6 mm, vias 0 -> 2
- net Net-(D1-Pad1): track 0.00 -> 16.9 mm, vias 0 -> 4
- net Net-(D1-Pad2): track 0.00 -> 14.8 mm
- net /speedPulse: track 0.00 -> 5.33 mm
- net Net-(SW1-Pad2): track 0.00 -> 3.81 mm
- net Net-(C4-Pad1): track 0.00 -> 3.29 mm
- net Net-(Q1-Pad3): track 0.00 -> 3.20 mm
- net +3V3: track 0.00 -> 2.26 mm
- net /EN_DYN: track 0.00 -> 2.18 mm
- net (no net): vias 0 -> 6
- added copper zone on B.Cu, net +BATT
- added copper zone on F.Cu, net +BATT
- added copper zone on F.Cu, net Net-(C4-Pad1)
- added copper zone on F.Cu, net Net-(D1-Pad1)

Commit message: top half is routed
Parts:
- C1, C3, D1, D2, D3, D4, R5: moved to B.Cu
- moved C1 13.4 mm to (167.6, 83.2), turned to 180 degrees
- moved R5 10.8 mm to (177.8, 94.0)
- moved D7 9.53 mm to (170.2, 79.4), turned to 180 degrees
- moved C2 8.84 mm to (182.2, 110.9), turned to 180 degrees
- moved R6 7.41 mm to (170.2, 76.8), turned to 180 degrees
- moved C3 5.43 mm to (178.4, 64.8), turned to 90 degrees
- moved D6 4.96 mm to (174.0, 79.4)
- moved U3 0.90 mm to (178.4, 64.1)
- moved U1 0.64 mm to (178.4, 88.3)
- moved Q1 0.63 mm to (188.6, 89.5)
- moved R3 0.63 mm to (191.8, 89.5)
Routing:
- net +3V3: track 2.26 -> 92.2 mm, vias 0 -> 5
- net /SDA: track 0.00 -> 63.7 mm, vias 0 -> 2
- net /SCL: track 0.00 -> 60.2 mm, vias 0 -> 1
- net /speedPulse: track 5.33 -> 32.0 mm, vias 0 -> 1
- net /EN_DYN: track 2.18 -> 26.1 mm, vias 0 -> 1
- net +BATT: track 34.3 -> 52.4 mm, vias 7 -> 9
- net GND: track 0.00 -> 9.77 mm, vias 0 -> 11
- net Net-(D3-Pad2): track 33.2 -> 27.0 mm, vias 4 -> 3
- net Net-(D5-Pad2): track 21.6 -> 16.4 mm, vias 2 -> 0
- net /prog_rst: track 0.00 -> 3.69 mm, vias 0 -> 1
- net Net-(D1-Pad1): track 16.9 -> 18.4 mm, vias 4 -> 2
- net Net-(C4-Pad1): track 3.29 -> 4.08 mm
- net Net-(Q1-Pad3): track 3.20 -> 3.84 mm
- net Net-(D1-Pad2): track 14.8 -> 14.7 mm, vias 0 -> 2
- net (no net): vias 6 -> 0
- added copper zone on B.Cu, net GND
- added copper zone on F.Cu, net GND
- removed copper zone on B.Cu, net +BATT

Commit message: das Schwein ist bestellt!
Parts:
- removed J2: Conn_01x05_Male, Connector_JST:JST_XH_S5B-XH-A-1_1x05_P2.50mm_Horizontal
- removed SW1: JMP, Connector_PinHeader_2.54mm:PinHeader_1x02_P2.54mm_Horizontal
- added C5: 10u, Capacitor_SMD:C_0603_1608Metric, B.Cu at (178.1, 89.5)
- added C6: 1u, Capacitor_SMD:C_0805_2012Metric, B.Cu at (173.4, 117.5)
- added L1: DO1608C-223MLB, myStuff:DO1608, B.Cu at (173.6, 86.4)
- added R8: 13k3, Resistor_SMD:R_0805_2012Metric, B.Cu at (182.9, 87.6)
- added R9: 41k2, Resistor_SMD:R_0805_2012Metric, B.Cu at (182.9, 89.9)
- C1: value 1u -> 10u; footprint Capacitor_SMD:C_0805_2012Metric -> Capacitor_SMD:C_0603_1608Metric
- D5, D6, D7, Q1, Q2, R1, R2, R3, R4, R6, R7, U3: moved to B.Cu
- U1: value DCDC_mod -> TPS560200; footprint myStuff:ebay_dcdc -> Package_TO_SOT_SMD:SOT-23-5
- moved R7 29.5 mm to (174.0, 94.0)
- moved U5 17.8 mm to (168.9, 99.7), turned to 270 degrees
- moved R1 11.5 mm to (191.1, 84.5)
- moved C1 11.3 mm to (178.1, 87.6), turned to 0 degrees
- moved R6 10.9 mm to (163.8, 85.7)
- moved D6 8.82 mm to (169.5, 87.0), turned to 90 degrees
- moved D7 8.26 mm to (167.0, 87.0), turned to 270 degrees
- moved D5 6.48 mm to (190.5, 81.9)
- moved C3 5.18 mm to (174.0, 67.4), turned to 180 degrees
- moved U1 4.10 mm to (180.0, 84.5), turned to 0 degrees
- moved Q2 4.02 mm to (188.6, 76.8), turned to 0 degrees
- moved R2 3.70 mm to (186.7, 82.5), turned to 270 degrees
- moved Q1 1.91 mm to (188.6, 87.6), turned to 90 degrees
- moved R3 1.91 mm to (191.8, 87.6)
- moved R4 1.27 mm to (183.5, 64.1), turned to 90 degrees
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Connections:
- R4 pad 1: Net-(C4-Pad1) -> +BATT
- R4 pad 2: +BATT -> Net-(C4-Pad1)
- TP1 pad 1: Net-(TP1-Pad1) -> /prog_btn
- U1 pad 1: +3V3 -> (no net)
- U1 pad 3: +BATT -> Net-(L1-Pad1)
- U1 pad 4: Net-(SW1-Pad2) -> +BATT
- U2 pad 10: Net-(J2-Pad4) -> (no net)
- U2 pad 11: Net-(J2-Pad5) -> /EN1
- U2 pad 12: Net-(TP2-Pad1) -> /EN0
- U2 pad 16: /EN0 -> (no net)
- U2 pad 23: Net-(TP1-Pad1) -> /speedPulse
- U2 pad 24: /speedPulse -> Net-(TP2-Pad1)
- U2 pad 26: /EN1 -> Net-(TP3-Pad1)
- U2 pad 29: /EN2 -> (no net)
- U2 pad 33: Net-(J2-Pad1) -> (no net)
- U2 pad 36: Net-(J2-Pad2) -> (no net)
- U2 pad 37: Net-(J2-Pad3) -> (no net)
- U2 pad 4: (no net) -> /EN2
- U2 pad 8: Net-(TP3-Pad1) -> Net-(TP4-Pad1)
- U2 pad 9: Net-(TP4-Pad1) -> (no net)
- U3 pad 7: +BATT -> Net-(C4-Pad1)
- U3 pad 8: Net-(C4-Pad1) -> +BATT
Routing:
- net /prog_rst: track 3.69 -> 50.3 mm, vias 1 -> 4
- net Net-(TP4-Pad1): track 0.00 -> 26.9 mm, vias 0 -> 2
- net /prog_rx: track 0.00 -> 23.2 mm, vias 0 -> 1
- net /prog_tx: track 0.00 -> 21.4 mm, vias 0 -> 1
- net /prog_btn: track 0.00 -> 18.2 mm, vias 0 -> 1
- net /EN0: track 0.00 -> 15.8 mm, vias 0 -> 2
- net +BATT: track 52.4 -> 67.8 mm, vias 9 -> 11
- net +3V3: track 92.2 -> 105.9 mm, vias 5 -> 7
- net Net-(D1-Pad1): track 18.4 -> 30.6 mm
- net Net-(TP3-Pad1): track 0.00 -> 11.3 mm, vias 0 -> 2
- net Net-(TP2-Pad1): track 0.00 -> 9.20 mm, vias 0 -> 1
- net Net-(D3-Pad2): track 27.0 -> 35.1 mm
- net Net-(D5-Pad2): track 16.4 -> 8.38 mm
- net /SCL: track 60.2 -> 67.5 mm, vias 1 -> 2
- net /EN1: track 0.00 -> 6.63 mm, vias 0 -> 1
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- added copper zone on B.Cu, net +3V3
- added copper zone on B.Cu, net Net-(C4-Pad1)
- added copper zone on B.Cu, net Net-(L1-Pad1)
- removed copper zone on F.Cu, net Net-(C4-Pad1)
- removed copper zone on F.Cu, net Net-(D1-Pad1)
Other:
- board text added: "+"
- board text added: "-"
- board text added: "BAT"
- board text added: "DYN"
- board text added: "EN"
- board text added: "OUT0"
- board text added: "OUT1"
- board text added: "OUT2"
