File: PCB2/velogen2.kicad_pcb (KiCad board)
At the start: 2 copper layers, 35 x 70 mm, 39 parts, among them J1 DYN, J3 AUX0, J4 AUX1, J5 AUX2, J6 BAT, Q1 BSS123, Q2 DMP10H400SE, U1 TPS560200, U2 ESP32-WROOM-32, U3 INA219BxD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

Commit message: cad: tune the PCB shell, add oled spacer
Parts:
- R8: value 13k3 -> 15k
- R9: value 41k2 -> 47k
